Commit message: joint correction

File: rtb-data/rtbdata/xacro/mg400_description/urdf/mg400 copy.urdf (robot description, URDF)
Before this commit: robot mg400_description, 5 links, 4 joints
Links:
- added link fake_link
- added link link2_2, mass 0.0662546292985346; collision mesh filename=package://mg400_description/meshes/link2_2.STL; visual mesh filename=package://mg400_description/meshes/link2_2.STL
- added link link3_2, mass 0.0366692789294813; collision mesh filename=package://mg400_description/meshes/link3_2.STL; visual mesh filename=package://mg400_description/meshes/link3_2.STL
- added link link4_2, mass 0.0453569016333092; collision mesh filename=package://mg400_description/meshes/link4_2.STL; visual mesh filename=package://mg400_description/meshes/link4_2.STL
- added link link5, mass 0.0965276919819365; collision mesh filename=package://mg400_description/meshes/link5.STL; visual mesh filename=package://mg400_description/meshes/link5.STL
Joints:
- added joint j2_2: type revolute, parent link1, child link2_2, origin xyz=0.00452885682964267 -0.0305 0.141500000000001 rpy=0 0 0, axis 0 1 0, limit lower=-3.14 upper=3.14 effort=0 velocity=0, mimic joint=j2
- added joint j3_1: type revolute, parent fake_link, child link3_1, axis 0 1 0, limit lower=-3.14 upper=3.14 effort=0 velocity=0, mimic joint=j3_2
- added joint j3_2: type revolute, parent link2_2, child link3_2, origin xyz=-0.00105049750546494 0.00649999999999986 0.174996846985851 rpy=0 0 0, axis 0 1 0, limit lower=-3.14 upper=3.14 effort=0 velocity=0, mimic joint=j2_2 multiplier=-1
- added joint j4: type revolute, parent link4_1, child link5, origin xyz=0.0659996239003897 0.0170000000000371 0.031000800715573 rpy=0 0 0, axis -1.19408295462994E-05 0 0.999999999928708, limit lower=-3.14 upper=3.14 effort=0 velocity=0
- added joint j4_2: type revolute, parent link3_2, child link4_2, origin xyz=0.0678965856063864 0.000500000000000073 0.0119719999403219 rpy=0 0 0, axis 0 1 0, limit lower=-3.14 upper=3.14 effort=0 velocity=0, mimic joint=j3
- joint j3: child link3_1 -> fake_link
